File: KiCad/Keyboard.sch (KiCad schematic (older format))
At the start: 77 parts, among them J1 USB_mini_micro_B, K1 KEYSW, K10 KEYSW, K11 KEYSW, K12 KEYSW, K13 KEYSW, K14 KEYSW, K15 KEYSW, K16 KEYSW, K17 KEYSW, K18 KEYSW, K19 KEYSW, K2 KEYSW, K20 KEYSW, K21 KEYSW, K22 KEYSW, K3 KEYSW, K4 KEYSW, K5 KEYSW, K6 KEYSW, K7 KEYSW, K8 KEYSW, K9 KEYSW, SW1 SW_PUSH, U1 ATMEGA32U4, X1 XTAL_GND

Commit message: Completed COl connectons an UG and KG LEDS started RE LED connections
Parts:
- removed D? (x13): WS2812, LED_SMD:LED_WS2812_PLCC6_5.0x5.0mm_P1.6mm, symbol LED:WS2812
- added KG1, KG10, KG11, KG12, KG13, KG14, KG15, KG16, KG17, KG18, KG19, KG2, KG20, KG21, KG22, KG3, KG4, KG5, KG6, KG7, KG8, KG9, UG1, UG10, UG11, UG12, UG13, UG14, UG2, UG3, UG4, UG5, UG6, UG7, UG8, UG9: WS2812B, LED_SMD:LED_WS2812B_PLCC4_5.0x5.0mm_P3.2mm, symbol LED:WS2812B
- added U? (x4): WS2811, symbol Driver_LED:WS2811
Connections:
- wire segments 186 -> 257
- no-connect marks 14 -> 13
Other:
- note added: "Key LEDs (KG1 - KG22)"
- note added: "Rotary Encoder LEDS (RE1 - RE4)"
- note added: "Underglow LEDs (UG1 - UG14)"

Commit message: A bit closer, ran out of pins on MCU ugh!!
Parts:
- added RE1, RE2, RE3, RE4: ENCODER-RGB-SWITCH, ENCODER_LED_3, symbol SparkFun-Switches:ENCODER-RGB-SWITCH
- gave numbers to parts that had none: 4
Connections:
- net labels added: ledcontrol
- wire segments 257 -> 310
Other:
- note added: "Rotary Encoder LEDS (REG1 - REG4)"
- note removed: "Rotary Encoder LEDS (RE1 - RE4)"
- moved on the sheet: REG1, REG2, REG3, REG4

Commit message: all LEDs I think are setup, one question there in bold.
Parts:
- added C-KG1, C-KG10, C-KG11, C-KG12, C-KG13, C-KG14, C-KG15, C-KG16, C-KG17, C-KG18, C-KG19, C-KG2, C-KG20, C-KG21, C-KG22, C-KG3, C-KG4, C-KG5, C-KG6, C-KG7, C-KG8, C-KG9, C-REG1, C-REG2, C-REG3, C-REG4, C-UG1, C-UG10, C-UG11, C-UG12, C-UG13, C-UG14, C-UG2, C-UG3, C-UG4, C-UG5, C-UG6, C-UG7, C-UG8, C-UG9: 104, symbol Device:C
- added R-REG1, R-REG2, R-REG3, R-REG4: 100R, symbol Device:R
- added R-REG1, R-REG2, R-REG3, R-REG4: 33R, symbol Device:R
Connections:
- wire segments 310 -> 467
Other:
- note added: "R-REG4 is it needed"

Commit message: Changed to SMALL components
Parts:
- C-KG1, C-KG10, C-KG11, C-KG12, C-KG13, C-KG14, C-KG15, C-KG16, C-KG17, C-KG18, C-KG19, C-KG2, C-KG20, C-KG21, C-KG22, C-KG3, C-KG4, C-KG5, C-KG6, C-KG7, C-KG8, C-KG9, C-REG1, C-REG2, C-REG3, C-REG4, C-UG1, C-UG10, C-UG11, C-UG12, C-UG13, C-UG14, C-UG2, C-UG3, C-UG4, C-UG5, C-UG6, C-UG7, C-UG8, C-UG9: symbol Device:C -> Device:C_Small
- C10, C9: renamed from C?; symbol Device:C -> Device:C_Small
- C3, C4, C5, C6: value .1u -> 104
- D1, D10, D11, D12, D13, D14, D15, D16, D17, D18, D19, D2, D20, D21, D22, D3, D4, D5, D6, D7, D8, D9: symbol Device:D -> Device:D_Small
- R-REG1, R-REG2, R-REG3, R-REG4, R1, R2, R3, R4: symbol Device:R -> Device:R_Small
- R-VREG1: renamed from R-REG1; symbol Device:R -> Device:R_Small
- R-VREG2: renamed from R-REG2; symbol Device:R -> Device:R_Small
- R-VREG3: renamed from R-REG3; symbol Device:R -> Device:R_Small
- R-VREG4: renamed from R-REG4; symbol Device:R -> Device:R_Small
- gave numbers to parts that had none: 2
Connections:
- wire segments 467 -> 474
- no-connect marks 13 -> 18
Other:
- moved on the sheet: C3, C4, C5, C6, C7, J2, K1, K10, K11, K12, K13, K14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

Commit message: small changes
Connections:
- net SCL: now reaches U1.18 (PD0/INT0)
- net SCL: now also U2.2 (SCL)
- net SDA: now reaches U1.19 (PD1/INT1)
- net SDA: now also U2.3 (SDA)
Other:
- moved on the sheet: C1, C2
Changed lines of the file:
@@
 L Device:C_Small C1
 U 1 1 5EC134E7
-P 1800 3150
-F 0 "C1" H 1892 3196 50  0000 L CNN
-F 1 "22p" H 1892 3105 50  0000 L CNN
-F 2 "" H 1800 3150 50  0001 C CNN
-F 3 "~" H 1800 3150 50  0001 C CNN
-	1    1800 3150
+P 1800 3100
+F 0 "C1" H 1892 3146 50  0000 L CNN
+F 1 "22p" H 1892 3055 50  0000 L CNN
+F 2 "" H 1800 3100 50  0001 C CNN
+F 3 "~" H 1800 3100 50  0001 C CNN
+	1    1800 3100
 	1    0    0    -1
 $EndComp
@@
 L Device:C_Small C2
 U 1 1 5EC13D53
-P 2400 3150
-F 0 "C2" H 2492 3196 50  0000 L CNN
-F 1 "22p" H 2492 3105 50  0000 L CNN
-F 2 "" H 2400 3150 50  0001 C CNN
-F 3 "~" H 2400 3150 50  0001 C CNN
-	1    2400 3150
+P 2400 3100
+F 0 "C2" H 2492 3146 50  0000 L CNN
+F 1 "22p" H 2492 3055 50  0000 L CNN
+F 2 "" H 2400 3100 50  0001 C CNN
+F 3 "~" H 2400 3100 50  0001 C CNN
+	1    2400 3100
 	1    0    0    -1
 $EndComp
@@
 L keyboardparts:GND #PWR0101
 U 1 1 5EC16423
-P 2100 3550
-F 0 "#PWR0101" H 2100 3600 20  0001 C CNN
-F 1 "GND" H 2100 3609 30  0000 C CNN
-F 2 "" H 2100 3550 60  0000 C CNN
-F 3 "" H 2100 3550 60  0000 C CNN
-	1    2100 3550
+P 2100 3200
+F 0 "#PWR0101" H 2100 3250 20  0001 C CNN
+F 1 "GND" H 2100 3259 30  0000 C CNN
+F 2 "" H 2100 3200 60  0000 C CNN
+F 3 "" H 2100 3200 60  0000 C CNN
+	1    2100 3200
 	1    0    0    -1
 $EndComp
@@
 	1800 2750 1800 2900
 Wire Wire Line
-	1800 3050 1800 2900
+	1800 3000 1800 2900
 Connection ~ 1800 2900
 Wire Wire Line
-	1800 3250 1800 3550
-Wire Wire Line
-	1800 3550 2100 3550
+	1800 3200 2100 3200
 Wire Wire Line
 	3050 2850 2400 2850
@@
 	2400 2850 2400 2900
 Wire Wire Line
-	2400 2900 2400 3050
+	2400 2900 2400 3000
 Connection ~ 2400 2900
 Wire Wire Line
-	2400 3250 2400 3550
-Wire Wire Line
-	2400 3550 2100 3550
-Connection ~ 2100 3550
+	2400 3200 2100 3200
+Connection ~ 2100 3200
 Wire Wire Line
-	2100 3100 2100 3550
+	2100 3100 2100 3200
 $Comp
 L power:VCC #PWR0102
@@
 L power:VCC #PWR0104
 U 1 1 5EC238FE
-P 1250 2100
-F 0 "#PWR0104" H 1250 1950 50  0001 C CNN
-F 1 "VCC" V 1265 2227 50  0000 L CNN
-F 2 "" H 1250 2100 50  0001 C CNN
-F 3 "" H 1250 2100 50  0001 C CNN
-	1    1250 2100
+P 1350 2100
+F 0 "#PWR0104" H 1350 1950 50  0001 C CNN
+F 1 "VCC" V 1365 2227 50  0000 L CNN
+F 2 "" H 1350 2100 50  0001 C CNN
+F 3 "" H 1350 2100 50  0001 C CNN
+	1    1350 2100
 	0    -1   -1   0
 $EndComp
@@
 L keyboardparts:GND #PWR0105
 U 1 1 5EC23EF0
-P 750 2450
-F 0 "#PWR0105" H 750 2500 20  0001 C CNN
-F 1 "GND" H 750 2509 30  0000 C CNN
-F 2 "" H 750 2450 60  0000 C CNN
-F 3 "" H 750 2450 60  0000 C CNN
-	1    750  2450
-	1    0    0    -1
+P 1100 2450
+F 0 "#PWR0105" H 1100 2500 20  0001 C CNN
+F 1 "GND" H 1100 2509 30  0000 C TNN
+F 2 "" H 1100 2450 60  0000 C CNN
+F 3 "" H 1100 2450 60  0000 C CNN
+	1    1100 2450
+	0    1    1    0
 $EndComp
 $Comp
@@
 	1    0    0    -1
 $EndComp
-Wire Wire Line
-	1100 2450 750  2450
 $Comp
 L Device:R_Small R1
@@
 	1700 2450 1850 2450
 Wire Wire Line
-	1350 2100 1250 2100
-Wire Wire Line
 	1850 2100 1850 2450
 Wire Wire Line
@@
 NoConn ~ 3050 2250
 NoConn ~ 3050 2350
-NoConn ~ 3050 2950
-NoConn ~ 3050 3050
 NoConn ~ 3050 3150
 NoConn ~ 3050 3250
@@
 $EndComp
 $Comp
-L keyboardparts:GND #PWR0120
-U 1 1 5ECD6149
-P 7800 5300
-F 0 "#PWR0120" H 7800 5350 20  0001 C CNN
-F 1 "GND" V 7800 5329 30  0000 L CNN
-F 2 "" H 7800 5300 60  0000 C CNN
-F 3 "" H 7800 5300 60  0000 C CNN
-	1    7800 5300
-	0    1    1    0
-$EndComp
-Wire Wire Line
-	8000 5300 7800 5300
-$Comp
 L Device:C_Small C10
 U 1 1 5ECEAA5D
@@
 Wire Wire Line
 	5200 2350 5550 2350
+NoConn ~ 5200 3150
+NoConn ~ 5200 3050
+$Comp
+L keyboardparts:GND #PWR0120
+U 1 1 5ECD6149
+P 8000 5300
+F 0 "#PWR0120" H 8000 5350 20  0001 C CNN
+F 1 "GND" V 8000 5329 30  0000 L CNN
+F 2 "" H 8000 5300 60  0000 C CNN
+F 3 "" H 8000 5300 60  0000 C CNN
+	1    8000 5300
+	0    1    1    0
+$EndComp
+Text Label 7750 5100 0    50   ~ 0
+SCL
+Text Label 7750 5000 0    50   ~ 0
+SDA
+Wire Wire Line
+	7750 5000 8000 5000
+Wire Wire Line
+	7750 5100 8000 5100
+Text Label 2850 2950 0    50   ~ 0
+SCL
+Text Label 2850 3050 0    50   ~ 0
+SDA
+Wire Wire Line
+	2850 3050 3050 3050
+Wire Wire Line
+	2850 2950 3050 2950
 $EndSCHEMATC

Commit message: Got the envoder switches wired up
Parts:
- added D? (x4): D, symbol Device:D_Small
- added LS?: Speaker, symbol Device:Speaker
- added Q? (x5): 2N3904, Package_TO_SOT_THT:TO-92_Inline, symbol Transistor_BJT:2N3904
- added R?: 220R, symbol Device:R_Small
Connections:
- net ledcontrol is gone; now on net RGBMatrix: UG1.4 (DIN)
- net +5V: now also Q?.1 (E)
- net VCC: now also LS?.1
- net col1: now also Q?.3 (C), Q?.3 (C)
- net col7: now also Q?.3 (C), Q?.3 (C)
- net row3: now also D?.1 (K), D?.1 (K)
- net row5: now also D?.1 (K), D?.1 (K)
- net RGBMatrix: now reaches U1.25 (ICP1/PD4)
- net PWMSound: now reaches U1.26 (T1/PD6)
- net PWMSound: now also R?.2
- net ENC1_PB: now reaches RE1.3 (SW)
- net ENC1_PB: now also Q?.2 (B)
- net ENC2_PB: now reaches RE2.3 (SW)
- net ENC2_PB: now also Q?.2 (B)
- net ENC3_PB: now reaches RE3.3 (SW)
- net ENC3_PB: now also Q?.2 (B)
- net ENC4_PB: now reaches RE4.3 (SW)
- net ENC4_PB: now also Q?.2 (B)
- new net: LS?.2, Q?.3 (C)
- new net: Q?.2 (B), R?.1
- new net: D?.2 (A), Q?.1 (E) (x4)
- no-connect marks 18 -> 20
Other:
- note added: "Haptic Feedback"
- note added: "Keyboard"
- note added: "Sounds/Music"
- moved on the sheet: C1, C2, C8, D1, D10, D11, D12, D13, D14, D15, D16, D17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

Commit message: well out of pins.. no bluetooh yet
Parts:
- removed Q? (x5): 2N3904, Package_TO_SOT_THT:TO-92_Inline, symbol Transistor_BJT:2N3904
- added Q-ENC1, Q-ENC2, Q-ENC3, Q-ENC4, Q-SOUND1: PZT2222A, Package_TO_SOT_SMD:SOT-223-3_TabPin2, symbol Transistor_BJT:PZT2222A
- gave numbers to parts that had none: 6
Connections:
- net +5V: now also Q-SOUND1.3 (E)
- net ENC1_PB: now also Q-ENC1.1 (B)
- net ENC2_PB: now also Q-ENC2.1 (B)
- net ENC3_PB: now also Q-ENC3.1 (B)
- net ENC4_PB: now also Q-ENC4.1 (B)
- net RGBMatrix: now also KG1.4 (DIN); no longer UG1.4 (DIN)
- net col1: now also Q-ENC1.2 (C), Q-ENC3.2 (C)
- net col7: now also Q-ENC2.2 (C), Q-ENC4.2 (C)
- net Underglow: now reaches U1.1 (PE6/AIN0)
- net Underglow: now also UG1.4 (DIN)
- net ENC2_A: now reaches U1.10 (PB2/MOSI)
- net ENC2_A: now also RE2.A
- net ENC2_B: now reaches U1.11 (PB3/MISO)
- net ENC2_B: now also RE2.B
- net ENC3_A: now reaches U1.12 (PB7/~RTS)
- net ENC3_A: now also RE3.A
- net ENC3_B: now reaches U1.20 (PD2/RXD1)
- net ENC3_B: now also RE3.B
- net ENC4_A: now reaches U1.21 (PD3/TXD1)
- net ENC4_A: now also RE4.A
- net ENC4_B: now reaches U1.22 (PD5/XCK1)
- net ENC4_B: now also RE4.B
- net ENC1_A: now reaches U1.8 (PB0/SS)
- net ENC1_A: now also RE1.A
- net ENC1_B: now reaches U1.9 (PB1/SCK)
- net ENC1_B: now also RE1.B
- net at UG14.2 (DOUT): no longer KG1.4 (DIN)
- net at LS1.2: now also Q-SOUND1.2 (C)
- net at R-SOUND1.1: now also Q-SOUND1.1 (B)
- net at D-ENC1.2 (A): now also Q-ENC1.3 (E)
- net at D-ENC3.2 (A): now also Q-ENC3.3 (E)
- net at D-ENC2.2 (A): now also Q-ENC2.3 (E)
- net at D-ENC4.2 (A): now also Q-ENC4.3 (E)
- no-connect marks 20 -> 11

Commit message: lots of changes, and trying to get qmk done
Parts:
- removed C8: 1u, symbol Device:C_Small
- removed U1: ATMEGA32U4, symbol keyboardparts:ATMEGA32U4
- added C11: 1uF, symbol Device:C_Small
- added C12: 10pF, symbol Device:C_Small
- added J3: Conn_01x09_Female, symbol Connector:Conn_01x09_Female
- added J4: Conn_01x04_Female, symbol Connector:Conn_01x04_Female
- added LS2: Speaker, symbol Device:Speaker
- added Q-SOUND2: PZT2222A, Package_TO_SOT_SMD:SOT-223-3_TabPin2, symbol Transistor_BJT:PZT2222A
- added R-SOUND2: 220R, symbol Device:R_Small
- added SW_DIP1: SW_DIP_x08, symbol Switch:SW_DIP_x08
- added U1: AT90USB1287-MU, Package_DFN_QFN:QFN-64-1EP_9x9mm_P0.5mm_EP7.5x7.5mm, symbol MCU_Microchip_AVR:AT90USB1287-MU
- C1: value 22p -> 1uF
- C2: value 22p -> 10pF
- R1, R2: value 10k -> 22R
- R3, R4: value 22 -> 10k
- X1: value XTAL_GND -> 16Mhz
Connections:
- net +5V: now also C1.1, C10.2, R3.1, U2.8 (GND), C11.1, C12.1, J3.8 (Pin_8), J4.3 (Pin_3), Q-SOUND2.3 (E), SW_DIP1.10, SW_DIP1.11, SW_DIP1.12, SW_DIP1.13, SW_DIP1.14, SW_DIP1.15, SW_DIP1.16, SW_DIP1.9, U1.22 (GND), U1.53 (GND), U1.6 (UGND), U1.63 (GND), U1.65 (GND); no longer C1.2, R2.2
- net ENC1_A: now also U1.61 (PF0)
- net ENC1_B: now also U1.60 (PF1)
- net ENC2_A: now also U1.59 (PF2)
- net ENC2_B: now also U1.58 (PF3)
- net ENC3_A: now also U1.57 (PF4)
- net ENC3_B: now also U1.56 (PF5)
- net ENC4_A: now also U1.55 (PF6)
- net ENC4_B: now also U1.54 (PF7)
- net RGBMatrix: now also U1.32 (PD7)
- net SCL: now also J4.2 (Pin_2), U1.25 (PD0)
- net SDA: now also J4.1 (Pin_1), U1.26 (PD1)
- net Underglow: now also U1.31 (PD6)
- net VCC: now also C10.1, R4.2, U2.10 (VDD), J3.9 (Pin_9), J4.4 (Pin_4), LS2.1; no longer J1.1 (VUSB), R1.1
- net col1: now also U1.46 (PA5)
- net col2: now also U1.45 (PA6)
- net col3: now also U1.44 (PA7)
- net col4: now also U1.18 (PE4)
- net col5: now also U1.19 (PE5)
- net col6: now also U1.1 (PE6)
- net col7: now also U1.2 (PE7)
- net row1: now also U1.51 (PA0)
- net row2: now also U1.50 (PA1)
- net row3: now also U1.49 (PA2)
- net row4: now also U1.48 (PA3)
- net row5: now also U1.47 (PA4)
- net at SW1.2: now also R4.1, U1.20 (~RESET); no longer R1.2
- net at X1.1: now also C2.1, U1.24 (XTAL1); no longer C1.1
- net at X1.2: now also C12.2, U1.23 (XTAL2); no longer C2.1
- net at R3.2: now also U1.43 (PE2/~HWB)
- net at R2.1: now also U1.4 (D-)
- net at J1.2 (D-): now also R2.2; no longer R3.1
- net at J1.3 (D+): now also R1.1; no longer R4.1
- net at J1.4 (ID): now also U1.9 (PE3)
- net PWMSound renamed PWMSound1
- net PWMSound1: now also U1.15 (PB5)
- new net: C1.2, J1.1 (VUSB), U1.21 (VCC), U1.3 (UVCC), U1.52 (VCC), U1.64 (AVCC), U1.8 (VBUS)
- new net: SW_DIP1.8, U1.27 (PD2)
- new net: SW_DIP1.1, U1.35 (PC0)
- new net: SW_DIP1.2, U1.36 (PC1)
- new net: SW_DIP1.3, U1.37 (PC2)
- new net: SW_DIP1.4, U1.38 (PC3)
- new net: SW_DIP1.5, U1.39 (PC4)
- new net: SW_DIP1.6, U1.40 (PC5)
- new net: SW_DIP1.7, U1.42 (PC7)
- new net: R1.2, U1.5 (D+)
- new net: C11.2, U1.7 (UCAP)
- new net: Q-SOUND2.1 (B), R-SOUND2.1
- new net: LS2.2, Q-SOUND2.2 (C)
- new net BLECS: J3.4 (Pin_4), U1.14 (PB4)
- new net BLEIRQ: J3.5 (Pin_5), U1.28 (PD3)
- new net BLEReset: J3.7 (Pin_7), U1.29 (PD4)
- new net MISO: J3.2 (Pin_2), U1.13 (PB3)
- new net MOSI: J3.3 (Pin_3), U1.12 (PB2)
- new net PWMSound2: R-SOUND2.2, U1.41 (PC6)
- new net SCK: J3.1 (Pin_1), U1.11 (PB1)
- no-connect marks 11 -> 17
Other:
- note added: "Adafruit Bluetooth \n BLE SPI Friend\n"
- note added: "DIP SWITCH"
- note added: "ENCODERS"
- note added: "KEYBOARD"
- note added: "SCREEN\nSSD1306\n"
- moved on the sheet: C10, C3, C4, C5, C6, C7, C9, J2, LS1, Q-SOUND1, R-SOUND1, U2
