File: KiCad/Keyboard.sch (KiCad schematic (older format))
At the start: 174 parts, among them J1 USB_mini_micro_B, J2 Screw_Terminal_01x02, J3 Conn_01x09_Female, J4 Conn_01x04_Female, K1 KEYSW, K10 KEYSW, K11 KEYSW, K12 KEYSW, K13 KEYSW, K14 KEYSW, K15 KEYSW, K16 KEYSW, K17 KEYSW, K18 KEYSW, K19 KEYSW, K2 KEYSW, K20 KEYSW, K21 KEYSW, K22 KEYSW, K3 KEYSW, K4 KEYSW, K5 KEYSW, K6 KEYSW, K7 KEYSW, K8 KEYSW, K9 KEYSW, SW1 SW_PUSH, U1 AT90USB1287-MU, U2 DRV2605LDGS, X1 16Mhz

Commit message: all
Parts:
- C-KG1, C-KG10, C-KG11, C-KG12, C-KG13, C-KG14, C-KG15, C-KG16, C-KG17, C-KG18, C-KG19, C-KG2, C-KG20, C-KG21, C-KG22, C-KG3, C-KG4, C-KG5, C-KG6, C-KG7, C-KG8, C-KG9, C-REG1, C-REG2, C-REG3, C-REG4, C-UG1, C-UG10, C-UG11, C-UG12, C-UG13, C-UG2, C-UG3, C-UG4, C-UG5, C-UG6, C-UG7, C-UG8, C-UG9, C1, C10, C11, C12, C2, C3, C4, C5, C6, C7, C9: footprint (none) -> Capacitor_SMD:C_0201_0603Metric
- C-UG14, D-ENC1, D-ENC2, D-ENC3, D-ENC4, D1, D10, D11, D12, D13, D14, D15, D16, D17, D18, D19, D2, D20, D21, D22, D3, D4, D5, D6, D7, D8, D9: footprint (none) -> Diode_SMD:D_0201_0603Metric
- J1: footprint (none) -> Connector_USB:USB_Micro-B_Amphenol_10103594-0001LF_Horizontal
- J2, LS1, LS2: footprint (none) -> Connector_PinSocket_1.00mm:PinSocket_1x02_P1.00mm_Vertical_SMD_Pin1Left
- J3: value Conn_01x09_Female -> Bluetooth; footprint (none) -> Connector_PinSocket_1.00mm:PinSocket_1x04_P1.00mm_Vertical_SMD_Pin1Right
- J4: value Conn_01x04_Female -> Screen; footprint (none) -> Connector_PinSocket_1.00mm:PinSocket_1x03_P1.00mm_Vertical
- K1, K10, K11, K12, K13, K14, K15, K16, K17, K18, K19, K2, K20, K21, K22, K3, K4, K5, K6, K7, K8, K9: footprint (none) -> Button_Switch_Keyboard:SW_Cherry_MX_1.00u_Plate
- R-REG1, R-REG2, R-REG3, R-REG4, R-SOUND1, R-SOUND2, R-VREG1, R-VREG2, R-VREG3, R-VREG4, R1, R2, R3, R4: footprint (none) -> Resistor_SMD:R_0201_0603Metric
- RE1, RE2, RE3, RE4: footprint ENCODER_LED_3 -> Switches:ENCODER_LED_3
- REG1, REG2, REG3, REG4: footprint (none) -> Package_SO:SOP-8_3.9x4.9mm_P1.27mm
- SW1: footprint (none) -> Button_Switch_SMD:SW_DIP_SPSTx01_Slide_6.7x4.1mm_W6.73mm_P2.54mm_LowProfile_JPin
- SW_DIP1: footprint (none) -> Switches:DIPSWITCH-08
- X1: footprint (none) -> Crystal:Crystal_SMD_0603-2Pin_6.0x3.5mm
Connections:
- net +5V: no longer C-KG1.2, C-KG10.2, C-KG11.2, C-KG12.2, C-KG13.2, C-KG14.2, C-KG15.2, C-KG16.2, C-KG17.2, C-KG18.2, C-KG19.2, C-KG2.2, C-KG20.2, C-KG21.2, C-KG22.2, C-KG3.2, C-KG4.2, C-KG5.2, C-KG6.2, C-KG7.2, C-KG8.2, C-KG9.2, C-REG1.2, C-REG2.2, C-REG3.2, C-REG4.2, C-UG1.2, C-UG10.2, C-UG11.2, C-UG12.2, C-UG13.2, C-UG14.2, C-UG2.2, C-UG3.2, C-UG4.2, C-UG5.2, C-UG6.2, C-UG7.2, C-UG8.2, C-UG9.2, C1.1, C10.2, C11.1, C12.1, C2.2, C3.2, C4.2, C5.2, C6.2, C7.2, C9.2, J1.5 (GND), J1.6 (SHIELD), Q-SOUND1.3 (E), Q-SOUND2.3 (E), R3.1, RE1.C, RE2.C, RE3.C, RE4.C, REG1.4 (GND), REG2.4 (GND), REG3.4 (GND), REG4.4 (GND), SW1.1, SW_DIP1.10, SW_DIP1.11, SW_DIP1.12, SW_DIP1.13, SW_DIP1.14, SW_DIP1.15, SW_DIP1.16, SW_DIP1.9, U1.22 (GND), U1.53 (GND), U1.6 (UGND), U1.63 (GND), U1.65 (GND), U2.4 (IN/TRIG), U2.8 (GND), X1.3
- net ENC1_A: now also U1.60 (PF1); no longer U1.61 (PF0)
- net ENC1_B: now also U1.61 (PF0); no longer U1.60 (PF1)
- net ENC2_A: now also U1.54 (PF7); no longer U1.59 (PF2)
- net ENC2_B: now also U1.55 (PF6); no longer U1.58 (PF3)
- net ENC3_A: now also U1.58 (PF3); no longer U1.57 (PF4)
- net ENC3_B: now also U1.59 (PF2); no longer U1.56 (PF5)
- net ENC4_A: now also U1.56 (PF5); no longer U1.55 (PF6)
- net ENC4_B: now also U1.57 (PF4); no longer U1.54 (PF7)
- net GND: now also C-KG1.2, C-KG10.2, C-KG11.2, C-KG12.2, C-KG13.2, C-KG14.2, C-KG15.2, C-KG16.2, C-KG17.2, C-KG18.2, C-KG19.2, C-KG2.2, C-KG20.2, C-KG21.2, C-KG22.2, C-KG3.2, C-KG4.2, C-KG5.2, C-KG6.2, C-KG7.2, C-KG8.2, C-KG9.2, C-REG1.2, C-REG2.2, C-REG3.2, C-REG4.2, C-UG1.2, C-UG10.2, C-UG11.2, C-UG12.2, C-UG13.2, C-UG14.2, C-UG2.2, C-UG3.2, C-UG4.2, C-UG5.2, C-UG6.2, C-UG7.2, C-UG8.2, C-UG9.2, C1.1, C10.2, C11.1, C12.1, C2.2, C3.2, C4.2, C5.2, C6.2, C7.2, C9.2, J1.5 (GND), J1.6 (SHIELD), Q-SOUND1.3 (E), Q-SOUND2.3 (E), R3.1, RE1.C, RE2.C, RE3.C, RE4.C, REG1.4 (GND), REG2.4 (GND), REG3.4 (GND), REG4.4 (GND), SW1.1, SW_DIP1.10, SW_DIP1.11, SW_DIP1.12, SW_DIP1.13, SW_DIP1.14, SW_DIP1.15, SW_DIP1.16, SW_DIP1.9, U1.22 (GND), U1.53 (GND), U1.6 (UGND), U1.63 (GND), U1.65 (GND), U2.4 (IN/TRIG), U2.8 (GND), X1.3
- net at KG14.2 (DOUT): now also R-REG1.2; no longer KG15.4 (DIN)
- net at KG16.2 (DOUT): now also R-REG2.2; no longer KG17.4 (DIN)
- net at KG20.2 (DOUT): now also R-REG3.2; no longer KG21.4 (DIN)
- net at KG22.2 (DOUT): now also R-REG4.2; no longer R-REG4.1
- net at REG1.5 (DO): now also KG15.4 (DIN)
- net at REG1.6 (DIN): now also R-REG1.1; no longer R-REG1.2
- net at REG2.5 (DO): now also KG17.4 (DIN); no longer R-REG1.1
- net at REG2.6 (DIN): now also R-REG2.1; no longer R-REG2.2
- net at REG3.5 (DO): now also KG21.4 (DIN); no longer R-REG2.1
- net at REG3.6 (DIN): now also R-REG3.1; no longer R-REG3.2
- net at REG4.5 (DO): no longer R-REG3.1
- net at REG4.6 (DIN): now also R-REG4.1; no longer R-REG4.2
Other:
- moved on the sheet: C-KG15, C-KG16, C-KG17, C-KG18, C-KG19, C-KG20, C-KG21, C-KG22, C-REG1, C-REG2, C-REG3, C-REG4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
