File: KiCad/Keyboard.kicad_pcb (KiCad board)
At the start: 2 copper layers, 163.8 x 111.8 mm, 174 parts, among them J1 USB_mini_micro_B, J2 Screw_Terminal_01x02, J3 Bluetooth, J4 Screen, K1 KEYSW, K10 KEYSW, K11 KEYSW, K12 KEYSW, K13 KEYSW, K14 KEYSW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

Commit message: lots of changes
Parts:
- moved C-KG8 20.5 mm to (119.4, -8.89)
Routing:
- net GND: track 263.8 -> 1395.5 mm, vias 0 -> 2
- net VCC: track 1634.5 -> 1663.7 mm
- net Net-(D-ENC4-Pad2): track 0.00 -> 20.5 mm, vias 0 -> 1
- net Net-(D-ENC2-Pad2): track 0.00 -> 17.0 mm, vias 0 -> 1
- net (no net): track 1.52 -> 0.00 mm
Other:
- board size 163.8 x 111.8 mm -> 163.8 x 116.8 mm
- net class Default: clearance 0.2 -> 0.1778
- rule trace_clearance: 0.2 -> 0.1778
- rule trace_min: 0.2 -> 0.1524
- rule via_min_size: 0.4 -> 0.1524
